File: Tasmodul_USB-Dimmer.brd (EAGLE design)
At the start: 21 x 42 mm, 27 parts, among them IC1 REG1117, J2 61400416021, Q1 BC817-16SMD, Q2 5.8A/30V/35mΩ, X1 USB-A

Commit message: Cleaned up schematic Added SCH and GERBER Updated documentation
Parts:
- Q2: value 5.8A/30V/35mΩ -> DMN3404L-7
Changed lines of the file:
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@@
 <attribute name="VALUE" x="11.675" y="4.405" size="1.27" layer="28" rot="MR270"/>
 </element>
-<element name="Q2" library="SparkFun-DiscreteSemi" library_urn="urn:adsk.eagle:library:514" package="SOT23-3" package3d_urn="urn:adsk.eagle:package:38446/1" value="5.8A/30V/35mΩ" x="13.5" y="6" smashed="yes" rot="MR0">
+<element name="Q2" library="SparkFun-DiscreteSemi" library_urn="urn:adsk.eagle:library:514" package="SOT23-3" package3d_urn="urn:adsk.eagle:package:38446/1" value="DMN3404L-7" x="13.5" y="6" smashed="yes" rot="MR0">
 <attribute name="NAME" x="12.8" y="6.951" size="0.8" layer="26" font="vector" ratio="12" rot="MR0"/>
 <attribute name="PROD_ID" value="TRANS-12988" x="13.5" y="6" size="1.778" layer="28" rot="MR0" display="off"/>
